File: kicad/Kaylee.kicad_pcb (KiCad board)
At the start: 4 copper layers, 90 x 65 mm, 4 parts

Commit message: added the Capt'n
Parts:
- added C1: 220uF/35V, Capacitor_THT:CP_Radial_D10.0mm_P5.00mm, F.Cu at (68.0, 12.0)
- added C2: 220uF/35V, Capacitor_THT:CP_Radial_D10.0mm_P5.00mm, F.Cu at (79.0, 12.0)
- added C3: 100nF/50V, Capacitor_SMD:C_0805_2012Metric, F.Cu at (44.0, 24.0)
- added CM1: WE-SL5_7440640500, Kaylee:CMC_WE-SL5_7440640500, F.Cu at (31.0, 12.0)
- added CM2: WE-SL5_7440640500, Kaylee:CMC_WE-SL5_7440640500, F.Cu at (44.0, 12.0)
- added C_BEC1_IN: 100uF/50V, Capacitor_THT:CP_Radial_D10.0mm_P5.00mm, F.Cu at (69.0, 8.00)
- added C_BEC1_OUT: 100uF/50V, Capacitor_THT:CP_Radial_D10.0mm_P5.00mm, F.Cu at (70.0, 19.0)
- added C_BEC2_IN: 100uF/50V, Capacitor_THT:CP_Radial_D10.0mm_P5.00mm, F.Cu at (69.0, 28.0)
- added C_BEC2_OUT: 100uF/50V, Capacitor_THT:CP_Radial_D10.0mm_P5.00mm, F.Cu at (70.0, 39.0)
- added C_BEC_SV_IN: 100uF/50V, Capacitor_THT:CP_Radial_D10.0mm_P5.00mm, F.Cu at (69.0, 48.0)
- added C_BEC_SV_OUT: 100uF/50V, Capacitor_THT:CP_Radial_D10.0mm_P5.00mm, F.Cu at (70.0, 59.0)
- added C_DM1: 10uF/50V, Inductor_SMD:L_1210_3225Metric, F.Cu at (37.0, 24.0)
- added C_Y1: 4.7nF/250V_Y2, Capacitor_THT:C_Disc_D4.3mm_W1.9mm_P5.00mm, F.Cu at (22.0, 24.0)
- added C_Y2: 4.7nF/250V_Y2, Capacitor_THT:C_Disc_D4.3mm_W1.9mm_P5.00mm, F.Cu at (29.0, 24.0)
- added D1: SMBJ33CA, Diode_SMD:D_SMB, F.Cu at (14.0, 24.0)
- added D_I2C: PRTR5V0U2X, Package_TO_SOT_SMD:SOT-363_SC-70-6, F.Cu at (59.0, 54.0)
- added D_OR1: MBRD1045CT, Package_TO_SOT_SMD:TO-252-3_TabPin2, F.Cu at (77.5, 22.0)
- added D_OR2: MBRD1045CT, Package_TO_SOT_SMD:TO-252-3_TabPin2, F.Cu at (77.5, 42.0)
- added F1: FuseHolder_MAXI_150A, Kaylee:FuseHolder_MAXI_PCB, F.Cu at (56.0, 9.00)
- added FB_5V1: WE-742792612, Capacitor_SMD:C_0805_2012Metric, F.Cu at (63.0, 8.00)
- added FB_5V2: WE-742792612, Capacitor_SMD:C_0805_2012Metric, F.Cu at (63.0, 28.0)
- added FB_6V: WE-742792612, Capacitor_SMD:C_0805_2012Metric, F.Cu at (63.0, 48.0)
- added F_ESC1: FuseHolder_Mini_40A, Fuse:Fuseholder_Blade_Mini_Keystone_3568, F.Cu at (3.00, 40.5)
- added F_ESC2: FuseHolder_Mini_40A, Fuse:Fuseholder_Blade_Mini_Keystone_3568, F.Cu at (17.0, 40.5)
- added F_ESC3: FuseHolder_Mini_40A, Fuse:Fuseholder_Blade_Mini_Keystone_3568, F.Cu at (31.0, 40.5)
- added F_ESC4: FuseHolder_Mini_40A, Fuse:Fuseholder_Blade_Mini_Keystone_3568, F.Cu at (45.0, 40.5)
- added J_5V: NanoFit-4P_5V, Connector_Molex:Molex_Nano-Fit_105309-xx04_1x04_P2.50mm_Vertical, F.Cu at (83.5, 47.5)
- added J_6V: NanoFit-4P_6V, Connector_Molex:Molex_Nano-Fit_105309-xx04_1x04_P2.50mm_Vertical, F.Cu at (83.5, 55.5)
- added J_ALERT: JST-GH_2P_ALERT, Connector_JST:JST_GH_BM02B-GHS-TBT_1x02-1MP_P1.25mm_Vertical, F.Cu at (68.0, 60.0)
- added J_BATT: XT60PW-F, Connector_AMASS:AMASS_XT60PW-F_1x02_P7.20mm_Horizontal, F.Cu at (13.0, 19.0)
- added J_CHASSIS: M3_Lug, MountingHole:MountingHole_3.2mm_M3_Pad_Via, F.Cu at (5.00, 32.0)
- added J_ESC1: XT30PW-F_ESC1, Connector_AMASS:AMASS_XT30PW-F_1x02_P2.50mm_Horizontal, F.Cu at (8.00, 61.0)
- added J_ESC2: XT30PW-F_ESC2, Connector_AMASS:AMASS_XT30PW-F_1x02_P2.50mm_Horizontal, F.Cu at (22.0, 61.0)
- added J_ESC3: XT30PW-F_ESC3, Connector_AMASS:AMASS_XT30PW-F_1x02_P2.50mm_Horizontal, F.Cu at (36.0, 61.0)
- added J_ESC4: XT30PW-F_ESC4, Connector_AMASS:AMASS_XT30PW-F_1x02_P2.50mm_Horizontal, F.Cu at (50.0, 61.0)
- added J_I2C: JST-GH_4P_I2C, Connector_JST:JST_GH_BM04B-GHS-TBT_1x04-1MP_P1.25mm_Vertical, F.Cu at (62.0, 60.0)
- added J_PGND_BATT: M3_Lug, MountingHole:MountingHole_3.2mm_M3_Pad_Via, F.Cu at (5.00, 20.0)
- added J_SHLD_5V: M3_Lug, MountingHole:MountingHole_3.2mm_M3_Pad_Via, F.Cu at (87.0, 53.5)
- added J_SHLD_6V: M3_Lug, MountingHole:MountingHole_3.2mm_M3_Pad_Via, F.Cu at (85.5, 57.5)
- added J_SHLD_ALERT: M3_Lug, MountingHole:MountingHole_3.2mm_M3_Pad_Via, F.Cu at (65.5, 62.5)
- added J_SHLD_I2C: M3_Lug, MountingHole:MountingHole_3.2mm_M3_Pad_Via, F.Cu at (59.5, 62.5)
- added L_BEC1: WE-744314100_10uH, Inductor_SMD:L_1210_3225Metric, F.Cu at (77.0, 8.00)
- added L_BEC2: WE-744314100_10uH, Inductor_SMD:L_1210_3225Metric, F.Cu at (77.0, 28.0)
- added L_BEC3: WE-744314100_10uH, Inductor_SMD:L_1210_3225Metric, F.Cu at (77.0, 48.0)
- added Q_BATT_DSG: AON6556, Package_SO:SOIC-8_3.9x4.9mm_P1.27mm, F.Cu at (16.0, 33.0)
- added RS_1: 1mOhm_Kelvin_2512, Kaylee:R_Shunt_CSS2H_2512K, F.Cu at (8.00, 47.0)
- added RS_2: 1mOhm_Kelvin_2512, Kaylee:R_Shunt_CSS2H_2512K, F.Cu at (22.0, 47.0)
- added RS_3: 1mOhm_Kelvin_2512, Kaylee:R_Shunt_CSS2H_2512K, F.Cu at (36.0, 47.0)
- added RS_4: 1mOhm_Kelvin_2512, Kaylee:R_Shunt_CSS2H_2512K, F.Cu at (50.0, 47.0)
- added RS_MAIN: 1mOhm_Kelvin_2512, Kaylee:R_Shunt_CSS2H_2512K, F.Cu at (39.0, 33.0)
- added R_ALERT: 2.2k, Resistor_SMD:R_0402_1005Metric, F.Cu at (59.0, 59.0)
- added R_CHGND: 0R, Resistor_SMD:R_0402_1005Metric, F.Cu at (30.5, 33.0)
- added R_DSG_G: 10k, Resistor_SMD:R_0402_1005Metric, F.Cu at (25.0, 33.0)
- added R_FB1_1: 100k, Resistor_SMD:R_0402_1005Metric, F.Cu at (80.0, 7.50)
- added R_FB1_2: 22.1k, Resistor_SMD:R_0402_1005Metric, F.Cu at (84.5, 7.50)
- added R_FB2_1: 100k, Resistor_SMD:R_0402_1005Metric, F.Cu at (80.0, 24.5)
- added R_FB2_2: 22.1k, Resistor_SMD:R_0402_1005Metric, F.Cu at (84.5, 24.5)
- added R_FB6_1: 100k, Resistor_SMD:R_0402_1005Metric, F.Cu at (80.0, 44.5)
- added R_FB6_2: 30.1k, Resistor_SMD:R_0402_1005Metric, F.Cu at (84.5, 44.5)
- added U_BEC_5V_1: TPS54620RGYT, Package_DFN_QFN:Texas_RGP0020D_VQFN-20-1EP_4x4mm_P0.5mm_EP2.7x2.7mm, F.Cu at (84.0, 9.00)
- added U_BEC_5V_2: TPS54620RGYT, Package_DFN_QFN:Texas_RGP0020D_VQFN-20-1EP_4x4mm_P0.5mm_EP2.7x2.7mm, F.Cu at (84.0, 29.0)
- added U_BEC_6V: TPS54540DDAR, Package_SO:SOIC-8_3.9x4.9mm_P1.27mm, F.Cu at (84.0, 49.5)
- added U_IS1: INA226_0x40, Package_SO:MSOP-10_3x3mm_P0.5mm, F.Cu at (8.00, 53.0)
- added U_IS2: INA226_0x41, Package_SO:MSOP-10_3x3mm_P0.5mm, F.Cu at (22.0, 53.0)
- added U_IS3: INA226_0x42, Package_SO:MSOP-10_3x3mm_P0.5mm, F.Cu at (36.0, 53.0)
- added U_IS4: INA226_0x43, Package_SO:MSOP-10_3x3mm_P0.5mm, F.Cu at (50.0, 53.0)
- added U_IS_MAIN: INA226_0x44, Package_SO:MSOP-10_3x3mm_P0.5mm, F.Cu at (49.0, 33.0)
- H1, H2, H3, H4: value (none) -> M3; footprint MountingHole:MountingHole_3.2mm_M3_Pad_Via -> MountingHole:MountingHole_3.2mm_M3
Routing:
- added copper zone on In1.Cu, net PGND
- added copper zone on In2.Cu, net VBAT
