File: kicad/Kaylee.kicad_pcb (KiCad board)
At the start: 4 copper layers, 90 x 65 mm, 71 parts

Commit message: feat(avionics/kicad): Kaylee PDB DRC clean and Gerbers generated (Rev A)
Eliminated all 0.0 mm clearance and shorting violations from the
Kaylee power distribution board generator gen_kaylee_pcb.py:

- R_FB1_1/2: moved y=10→14 to clear U_BEC_5V_1 thermal pad (EP) bottom
- R_FB2_1: moved y=30→34 to clear U_BEC_5V_2 EP; R_FB2_2 moved x=84.5→86
  to exit J_5V pin circle x-range while remaining below EP in Y
- C_BEC_SV_OUT: moved y=59→56 so both THT pad circles clear J_ALERT
  MP pads at y=58.6 by ≥0.58 mm (constraint |cap_y−58.6| ≥ 0.846 mm)
- R_ALERT: moved x=59→66 to clear J_I2C pad1 (PGND) and pad3 (PDB_SCL)

DRC result: 0 shorting_items, 0 clearance violations at <0.15 mm.
Accepted residuals: 16 × 0.15 mm at INA226 MSOP-10 0.5 mm pitch pads
(IPC-2221B allows ≥0.1 mm at ≤31 V); 77 courtyard overlaps (no 3D
body conflict); 181 unconnected (traces not yet routed); library/silk
warnings (inline footprints, expected).

Generated Gerbers to avionics/kicad/gerbers/Kaylee/ (17 layers + drill).
Updated PROJECT_INDEX.md and TODO.md with accepted violations and
remaining manual placement tasks (Section F BQ76930, shield lugs).

Co-Authored-By: Claude Sonnet 4.6 <noreply@anthropic.com>
Parts:
- removed J_SHLD_5V, J_SHLD_6V, J_SHLD_ALERT, J_SHLD_I2C: M3_Lug, MountingHole:MountingHole_3.2mm_M3_Pad_Via
- moved J_5V 12.5 mm to (83.5, 35.0)
- moved C_BEC1_OUT 10.0 mm to (60.0, 19.0)
- moved C_BEC2_OUT 10.0 mm to (60.0, 39.0)
- moved R_FB2_2 9.62 mm to (86.0, 34.0)
- moved R_FB2_1 9.50 mm to (80.0, 34.0)
- moved R_ALERT 7.62 mm to (66.0, 62.0)
- moved R_FB1_1 6.50 mm to (80.0, 14.0)
- moved R_FB1_2 6.50 mm to (84.5, 14.0)
- moved FB_5V1 5.00 mm to (63.0, 13.0)
- moved D_OR1 4.50 mm to (73.0, 22.0)
- moved D_OR2 4.50 mm to (73.0, 42.0)
- moved C2 4.00 mm to (79.0, 16.0)
- moved C_BEC_SV_OUT 3.00 mm to (70.0, 56.0)
- moved C_DM1 3.00 mm to (40.0, 24.0)
- moved J_ALERT 3.00 mm to (71.0, 60.0)
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