File: kicad/Kaylee.kicad_pcb (KiCad board)
At the start: 4 copper layers, 90 x 65 mm, 67 parts

Commit message: chore(revision): synchronise avionics component designations to Rev R
Per CLAUDE.md: all components referenced as of the latest project revision.

Wash.md       — Rev A → Rev R; date 2026-06-02 → 2026-06-11;
                section "new in Rev A" → "Rev R baseline; introduced Rev A"
Kaylee.md     — title + Revision field Rev A → Rev R; date → 2026-06-11
XCVR-49MHZ-2.md — Rev A → Rev R; date 2026-06-02 → 2026-06-11
Zoë.md        — section "Rev A addition" → "Rev R baseline; introduced Rev A"
gen_kaylee.py — Reference line + silkscreen text Rev A → Rev R
gen_kaylee_pcb.py — silkscreen text Rev A → Rev R
Kaylee.kicad_pcb  — F.Fab silkscreen text "Kaylee Rev A" → "Kaylee Rev R"
Zoë.kicad_sch     — ETH_B comment "Rev Q addition" → "Rev R baseline"

All prior revision history preserved in parenthetical notes.

https://claude.ai/code/session_01Ke1YGpYGeikXWZswJmQKDh
Other:
- board text added: "Kaylee Rev R"
- board text removed: "Kaylee Rev A"
Changed lines of the file:
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@@
 		(stroke (width 0.05) (type default)) (layer "Edge.Cuts")
 )
-	(gr_text "Kaylee Rev A" (at 45.00 68.00 0) (layer "F.Fab")
+	(gr_text "Kaylee Rev R" (at 45.00 68.00 0) (layer "F.Fab")
 		(effects (font (size 1.5 1.5) (thickness 0.15)))
 )
