File: kicad/Zoë.kicad_sch (KiCad schematic)
At the start: 52 parts, among them SW1 SW_DIP_x02, X2Y_CAN 4.7nF_X2Y, X2Y_RS485 4.7nF_X2Y

Commit message: update emma
Other:
- note added: "ETH_B sub-circuit: EMI-hardened 10/100BASE-TX Ethernet PHY — Rev R baseline DP83825I PHY + HX1188NL magnetics + TPS62933 1.8V SMPS + PRTR5V0U2X TVS + SRF2012 CMC JST SM06B-GHS-TB-1MP connector J_ETH_B — RMII0 to PocketBeagle 2 AM6254"
Changed lines of the file:
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@@
     (pin "1")
   )
-  (comment 1 "ETH_B sub-circuit: EMI-hardened 10/100BASE-TX Ethernet PHY — Rev R baseline")
-  (comment 2 "DP83825I PHY + HX1188NL magnetics + TPS62933 1.8V SMPS + PRTR5V0U2X TVS + SRF2012 CMC")
-  (comment 3 "JST SM06B-GHS-TB-1MP connector J_ETH_B — RMII0 to PocketBeagle 2 AM6254")
+  (text "ETH_B sub-circuit: EMI-hardened 10/100BASE-TX Ethernet PHY — Rev R baseline\nDP83825I PHY + HX1188NL magnetics + TPS62933 1.8V SMPS + PRTR5V0U2X TVS + SRF2012 CMC\nJST SM06B-GHS-TB-1MP connector J_ETH_B — RMII0 to PocketBeagle 2 AM6254"
+    (at 300.00 118.00 0) (effects (font (size 1.27 1.27)) (justify left)))
   (symbol (lib_id "Conn_JST_GH_06P") (at 250.00 680.00 0)
     (unit 1) (exclude_from_sim no) (in_bom yes) (on_board yes) (dnp no)
