File: kicad/XCVR-49MHZ-2.kicad_pcb (KiCad board)
At the start: 4 copper layers, 55 x 35 mm, 69 parts, among them U1 ByA 100nF +3V3 U1-VDDA Bypass, U1 ByB 100nF +3V3 U1-VDD Bypass

Commit message: avionics: make Emma a stacking cape (P1/P2 + ETH + LoRa); Zoë passthrough rails
Implements the Rev R1 stack PocketBeagle -> Zoë -> Emma:

Emma (XCVR-49MHZ-2):
  * + PB2-P1/PB2-P2 2x18 sockets, wired pin-for-pin to the same nets as
    Zoë's headers (pass-through), making Emma a proper stacking cape.
  * + LoRa (RFM95W) moved from Zoë; wired to SPI1 (MISO/MOSI/CLK/CS_LORA)
    + LORA_RESETN, reached through the stack.
  * + Ethernet subsystem: ETH-PHY (ADIN1300) on RMII1 + PHY2_RSTN/INTRN
    (independent of Zoë's RMII0/PHY1), T-ETH (749010012A) and J-ETH on
    new EMMA_ETH_* MDI / EMMA_ETH_LINE_* nets. One ETH on Zoë, one on Emma.

Zoë:
  * - LoRa (now on Emma).
  * + PB2-P1-TOP / PB2-P2-TOP passthrough socket rails on the upper face,
    wired to the bottom-socket nets, so Emma stacks on top.

Net/component design only — new parts are placed at rough front-side
locations; dense 55x35 4-layer/both-side placement and routing are GUI
work (placement intentionally left for layout). LoRa 915 MHz antenna
routing on Emma and the now-redundant CAPE-B IF connector are follow-ups.

Co-Authored-By: Claude Opus 4.8 <noreply@anthropic.com>
Parts:
- added ETH-PHY: ADIN1300BCPZ, QFN-48-1EP_7x7mm_P0.5mm_EP5.65x5.65mm, F.Cu at (130.0, 118.0)
- added J-ETH: JST-GH-4P-ETH, JST_GH_4P, F.Cu at (147.0, 118.0)
- added LoRa: RFM95W, HOPERF_RFM9XW_SMD, F.Cu at (112.0, 118.0)
- added PB2-P1: PB2I-P1-2x18, 2x18_P1_Socket, F.Cu at (127.0, 103.5)
- added PB2-P2: PB2I-P2-2x18, 2x18_P2_Socket, F.Cu at (127.0, 131.5)
- added T-ETH: 749010012A, ETH_XFMR_8P_5x3.5mm, F.Cu at (140.0, 117.0)
Routing:
- net SPI1_CS_NOR: vias 0 -> 1
- net GND: vias 20 -> 18
- net +5V_FILT: vias 1 -> 2
