File: kicad/Emma.kicad_sch (KiCad schematic)
At the start: 6 parts, among them J1 JST_GH_06P_SHLD, J2 RPSMA_Edge

Commit message: update emma
Parts:
- removed CMC_CAN: SRF2012-100Y, Bourns_SRF2012, symbol SRF2012
- removed C_X2Y: 4.7nF X2Y, Capacitor_SMD:C_0402_1005Metric, symbol C
- removed D_TVS: PRTR5V0U2X, Package_TO_SOT_SMD:SOT-363_SC-88_MO-178CA, symbol PRTR5V0U2X
- removed FB1: 742792512, Inductor_SMD:L_0805_2012Metric, symbol Ferrite_Bead
- removed J1: JST_GH_06P_SHLD, Connector_JST:JST_GH_SM06B-GHS-TB_1x06-1MP_P1.25mm_Horizontal, symbol Conn_JST_GH_06P
- removed J2: RPSMA_Edge, Connector_Coaxial:SMA_Amphenol_132289_EdgeMount, symbol Conn_SMA
- added +3V 100n: 100nF X7R 0402 +3V3 HF Bypass, symbol S_+3V_100n
- added +3V 100u: 100uF 10V X5R 1210 +3V3 Bulk, symbol S_+3V_100u
- added +3V 10n: 10nF C0G 0402 +3V3 VHF 49MHz Bypass, symbol S_+3V_10n
- added +3V 10u: 10uF X5R 0805 +3V3 Mid-freq, symbol S_+3V_10u
- added +5V 100n: 100nF X7R 0402 +5V HF Bypass, symbol S_+5V_100n
- added +5V 100u: 100uF 10V X5R 1210 +5V Bulk, symbol S_+5V_100u
- added +5V Bead: 742792512, symbol S_+5V_Bead
- added 1.2k C: 10nF RX RC Bandpass 1200Hz Cap, symbol S_1.2k_C
- added 1.2k R: 13k Ohm RX RC Bandpass 1200Hz, symbol S_1.2k_R
- added 2.2k C: 10nF RX RC Bandpass 2200Hz Cap, symbol S_2.2k_C
- added 2.2k R: 7.2k Ohm RX RC Bandpass 2200Hz, symbol S_2.2k_R
- added 49M DDS: Si5351A-B-GT 49MHz DDS I2C Synthesiser, symbol S_49M_DDS
- added AFSK Cp: 1uF AFSK Audio Coupling DAC→PA, symbol S_AFSK_Cp
- added ANT CMC: SRF2012-100Y, symbol S_ANT_CMC
- added ANT RPSMA: RPSMA-EDGE-50R, symbol S_ANT_RPSMA
- added ANT TVS: PRTR5V0U2X, symbol S_ANT_TVS
- added C1 120p: 120pF C0G LPF Shunt-1, symbol S_C1_120p
- added C2 180p: 180pF C0G LPF Shunt-2, symbol S_C2_180p
- added C3 120p: 120pF C0G LPF Shunt-3, symbol S_C3_120p
- added CMP By: 100nF +3V3 U2B CMP Bypass, symbol S_CMP_By
- added C_INV: 100nF C0G 0402 INV1 VCC Bypass, symbol S_C_INV
- added C_MUX: 100nF C0G 0402 MUX1 VCC Bypass, symbol S_C_MUX
- added DAC By: 100nF +3V3 U2A DAC Bypass, symbol S_DAC_By
- added ETH-PHY: ADIN1300BCPZ, symbol S_ETH-PHY
- added GND X2Y: 4.7nF_X2Y_C0G, symbol S_GND_X2Y
- added INV1: SN74LVC1G04 SOT-23-5 3.3V UART_RX_F->SBUS_OUT, symbol S_INV1
- added J-ETH: JST-GH-4P-ETH, symbol S_J-ETH
- added L1 100n: 100nH Coilcraft-0805HQ-101J LPF Series-1, symbol S_L1_100n
- added L2 180n: 180nH Coilcraft-0805HQ-181J LPF Series-2, symbol S_L2_180n
- added L3 180n: 180nH Coilcraft-0805HQ-181J LPF Series-3, symbol S_L3_180n
- added LDO 3V3: MCP1703T-3302 LDO 3.3V 72dB-PSRR@100kHz, symbol S_LDO_3V3
- added LDO By: 100nF +3V3 U6 LDO Bypass, symbol S_LDO_By
- added LNA: MGA-82563 LNA 2.4dB NF 50-6000MHz, symbol S_LNA
- added LNA By: 100nF +3V3 U4 LNA Bypass, symbol S_LNA_By
- added LoRa: RFM95W, symbol S_LoRa
- added MUX1: SN74LVC1G157 SC-70-6 2:1MUX UART/SBUS Select, symbol S_MUX1
- added OSC By: 100nF +3V3 X1 TCXO Bypass, symbol S_OSC_By
- added PA 100mW: 2N3866 NPN BJT PA Class-AB Final 100mW, symbol S_PA_100mW
- added PA By: 100nF +5V U3 PA VCC Bypass, symbol S_PA_By
- added PA By2: 1nF U3B Collector RF Bypass, symbol S_PA_By2
- added PA Cb1: 100pF DDS-RF Coupling Cap to U3A, symbol S_PA_Cb1
- added PA Cb2: 100pF PA Interstage Bypass, symbol S_PA_Cb2
- added PA Drvr: MMBT2222A NPN BJT PA Class-A Driver, symbol S_PA_Drvr
- added PA Rb1: 10k Ohm U3A Base Bias Resistor, symbol S_PA_Rb1
- added PA Rb2: 1k Ohm U3B Base Bias Resistor, symbol S_PA_Rb2
- added PA Rc1: 100 Ohm U3A Collector Load, symbol S_PA_Rc1
- added PA Re: 10 Ohm U3B Emitter Degeneration, symbol S_PA_Re
- added PB2-P1: PB2I-P1-2x18, symbol S_PB2-P1
- added PB2-P2: PB2I-P2-2x18, symbol S_PB2-P2
- added PGND 10n: 10nF C0G 0402 GND-PGND Moat Bridge, symbol S_PGND_10n
- added PTT Bead: 742792510 0402 Ferrite Bead 600Ohm@100MHz, symbol S_PTT_Bead
- added RSSI Hi: 10k Ohm RSSI Scale Upper, symbol S_RSSI_Hi
- added RSSI Lo: 10k Ohm RSSI Scale Lower, symbol S_RSSI_Lo
- added RSSI_CBY: 100nF RSSI_CMP VCC Bypass, symbol S_RSSI_CBY
- added RSSI_CMP: LMV331 RSSI Carrier-Detect Comparator, symbol S_RSSI_CMP
- added RSSI_RH: 100k RSSI DCD Threshold Upper, symbol S_RSSI_RH
- added RSSI_RL: 100k RSSI DCD Threshold Lower, symbol S_RSSI_RL
- added RX Bead: 742792510 0402 Ferrite Bead 600Ohm@100MHz, symbol S_RX_Bead
- added RX Demod: LM393 Comparator RX-AFSK Demodulator, symbol S_RX_Demod
- added R_MODE: 10k Ohm MODE_SEL Pull-Down UART=default, symbol S_R_MODE
- added S1: SPST-SMD OPEN=UART CLOSED=SBUS, symbol S_S1
- added SMA ESD: SMAJ5.0A Bidirectional TVS 5V Antenna ESD, symbol S_SMA_ESD
- added SW By: 100nF +3V3 U5 Switch Bypass, symbol S_SW_By
- added T-ETH: 749010012A, symbol S_T-ETH
- added T/R Sw: PE4259-63 SPDT TX/RX Switch ≥35dB isolation, symbol S_T_R_Sw
- added TCXO 25M: TG2520SMN 25MHz TCXO ±0.5ppm, symbol S_TCXO_25M
- added TX Bead: 742792510 0402 Ferrite Bead 600Ohm@100MHz, symbol S_TX_Bead
- added TX DAC: MCP4921 12-bit SPI DAC TX-AFSK Audio, symbol S_TX_DAC
- added Th Hi: 10k Ohm LM393 Threshold Upper, symbol S_Th_Hi
- added Th Lo: 10k Ohm LM393 Threshold Lower, symbol S_Th_Lo
- added U1 ByA: 100nF +3V3 U1-VDDA Bypass, symbol S_U1_ByA
- added U1 ByB: 100nF +3V3 U1-VDD Bypass, symbol S_U1_ByB
- added UART CMC: SRF2012-100Y CMC UART TX/RX Pair 10uH, symbol S_UART_CMC
- added UART TVS: PRTR5V0U2X Dual TVS 5.5V UART-TX/RX ESD, symbol S_UART_TVS
Connections:
- net +5V: now also +5V Bead.1 (+5V), PB2-P1.35 (+5V), PB2-P2.35 (+5V)
- net GND: now also +3V 100n.2 (GND), +3V 100u.2 (GND), +3V 10n.2 (GND), +3V 10u.2 (GND), +5V 100n.2 (GND), +5V 100u.2 (GND), 1.2k C.2 (GND), 2.2k C.2 (GND), 49M DDS.2 (GND), 49M DDS.4 (GND), 49M DDS.5 (GND), 49M DDS.9 (GND), ANT RPSMA.2 (GND), ANT RPSMA.3 (GND), ANT TVS.1 (GND), ANT TVS.3 (GND), ANT TVS.4 (GND), ANT TVS.6 (GND), C1 120p.2 (GND), C2 180p.2 (GND), C3 120p.2 (GND), CMP By.2 (GND), C_INV.2 (GND), C_MUX.2 (GND), DAC By.2 (GND), ETH-PHY.10 (GND), ETH-PHY.11 (GND), ETH-PHY.12 (GND), ETH-PHY.3 (GND), ETH-PHY.49 (GND), ETH-PHY.6 (GND), GND X2Y.1 (GND), GND X2Y.2 (GND), INV1.2 (GND), LDO 3V3.2 (GND), LDO 3V3.5 (GND), LDO By.2 (GND), LNA By.2 (GND), LNA.5 (GND), LNA.6 (GND), LoRa.1 (GND), LoRa.10 (GND), LoRa.8 (GND), MUX1.2 (GND), OSC By.2 (GND), PA 100mW.2 (GND), PA By.2 (GND), PA By2.2 (GND), PA Cb2.2 (GND), PA Drvr.2 (GND), PA Re.2 (GND), PB2-P1.1 (GND), PB2-P1.2 (GND), PB2-P1.36 (GND), PB2-P2.36 (GND), PGND 10n.1 (GND), PGND 10n.2 (GND), RSSI Lo.2 (GND), RSSI_CBY.2 (GND), RSSI_CMP.4 (GND), RSSI_RL.2 (GND), RX Demod.4 (GND), RX Demod.5 (GND), R_MODE.2 (GND), SMA ESD.2 (GND), SW By.2 (GND), T/R Sw.2 (GND), T/R Sw.6 (GND), TCXO 25M.2 (GND), TX DAC.5 (GND), TX DAC.8 (GND), Th Hi.2 (GND), Th Lo.2 (GND), U1 ByA.2 (GND), U1 ByB.2 (GND), UART TVS.1 (GND), UART TVS.3 (GND), UART TVS.4 (GND), UART TVS.6 (GND)
- net PTT_N: now also PB2-P2.1 (PTT_N), PTT Bead.1 (PTT_N), PTT Bead.2 (PTT_N), T/R Sw.4 (PTT_N)
- new net +3V3: +3V 100n.1 (+3V3), +3V 100u.1 (+3V3), +3V 10n.1 (+3V3), +3V 10u.1 (+3V3), 49M DDS.1 (+3V3), 49M DDS.10 (+3V3), CMP By.1 (+3V3), C_INV.1 (+3V3), C_MUX.1 (+3V3), DAC By.1 (+3V3), INV1.4 (+3V3), LDO 3V3.3 (+3V3), LDO 3V3.4 (+3V3), LDO By.1 (+3V3), LNA By.1 (+3V3), LNA.4 (+3V3), MUX1.4 (+3V3), OSC By.1 (+3V3), PB2-P1.33 (+3V3), PB2-P1.34 (+3V3), RSSI_CBY.1 (+3V3), RSSI_CMP.2 (+3V3), RSSI_RH.1 (+3V3), RX Demod.2 (+3V3), S1.1 (+3V3), SW By.1 (+3V3), TCXO 25M.1 (+3V3), TCXO 25M.4 (+3V3), TX DAC.1 (+3V3), TX DAC.6 (+3V3), Th Hi.1 (+3V3), U1 ByA.1 (+3V3), U1 ByB.1 (+3V3)
- new net +5V_FILT: +5V 100n.1 (+5V_FILT), +5V 100u.1 (+5V_FILT), +5V Bead.2 (+5V_FILT), LDO 3V3.1 (+5V_FILT), PA By.1 (+5V_FILT), PA Rb1.1 (+5V_FILT), PA Rc1.1 (+5V_FILT)
- new net AFSK_IN: AFSK Cp.2 (AFSK_IN), RX Demod.1 (AFSK_IN)
- new net AFSK_OUT: AFSK Cp.1 (AFSK_OUT), TX DAC.7 (AFSK_OUT)
- new net ANT: ANT CMC.1 (ANT), ANT CMC.2 (ANT), ANT RPSMA.1 (ANT), ANT TVS.2 (ANT), SMA ESD.1 (ANT)
- new net CAN_STB: PB2-P1.12 (CAN_STB)
- new net COMP_IN: 1.2k C.1 (COMP_IN), 1.2k R.2 (COMP_IN), 2.2k C.1 (COMP_IN), 2.2k R.2 (COMP_IN), RX Demod.3 (COMP_IN), Th Lo.1 (COMP_IN)
- new net DDS_CLK: 49M DDS.6 (DDS_CLK), TX DAC.3 (DDS_CLK)
- new net DDS_DAT: 49M DDS.7 (DDS_DAT), TX DAC.4 (DDS_DAT)
- new net DDS_FSYNC: TX DAC.2 (DDS_FSYNC)
- new net DDS_RF: 49M DDS.3 (DDS_RF), PA Cb1.1 (DDS_RF), PA Drvr.1 (DDS_RF), PA Rb1.2 (DDS_RF)
- new net EMMA_ETH_LINE_RXN: J-ETH.4 (EMMA_ETH_LINE_RXN), T-ETH.8 (EMMA_ETH_LINE_RXN)
- new net EMMA_ETH_LINE_RXP: J-ETH.3 (EMMA_ETH_LINE_RXP), T-ETH.7 (EMMA_ETH_LINE_RXP)
- new net EMMA_ETH_LINE_TXN: J-ETH.2 (EMMA_ETH_LINE_TXN), T-ETH.6 (EMMA_ETH_LINE_TXN)
- new net EMMA_ETH_LINE_TXP: J-ETH.1 (EMMA_ETH_LINE_TXP), T-ETH.5 (EMMA_ETH_LINE_TXP)
- new net EMMA_ETH_RXN: ETH-PHY.5 (EMMA_ETH_RXN), T-ETH.4 (EMMA_ETH_RXN)
- new net EMMA_ETH_RXP: ETH-PHY.4 (EMMA_ETH_RXP), T-ETH.3 (EMMA_ETH_RXP)
- new net EMMA_ETH_TXN: ETH-PHY.2 (EMMA_ETH_TXN), T-ETH.2 (EMMA_ETH_TXN)
- new net EMMA_ETH_TXP: ETH-PHY.1 (EMMA_ETH_TXP), T-ETH.1 (EMMA_ETH_TXP)
- new net GND2_ETH: ETH-PHY.21 (GND2_ETH), ETH-PHY.22 (GND2_ETH), ETH-PHY.25 (GND2_ETH), ETH-PHY.34 (GND2_ETH), ETH-PHY.36 (GND2_ETH)
- new net I2C0_SCL: PB2-P1.4 (I2C0_SCL)
- new net I2C0_SDA: PB2-P1.3 (I2C0_SDA)
- new net LOAD_CELL_DOUT: PB2-P2.7 (LOAD_CELL_DOUT)
- new net LOAD_CELL_SCK: PB2-P2.8 (LOAD_CELL_SCK)
- new net LORA_DIO0: PB2-P1.20 (LORA_DIO0)
- new net LORA_RESETN: LoRa.6 (LORA_RESETN), PB2-P1.19 (LORA_RESETN)
- new net MCAN1_RX: PB2-P1.13 (MCAN1_RX)
- new net MCAN1_TX: PB2-P1.14 (MCAN1_TX)
- new net MDC: ETH-PHY.19 (MDC), PB2-P2.18 (MDC)
- new net MDIO: ETH-PHY.18 (MDIO), PB2-P2.17 (MDIO)
- new net MODE_SEL: MUX1.5 (MODE_SEL), R_MODE.1 (MODE_SEL), S1.2 (MODE_SEL)
- new net PA_EMIT: PA Re.1 (PA_EMIT)
- new net PA_INT: PA 100mW.1 (PA_INT), PA Cb1.2 (PA_INT), PA Cb2.1 (PA_INT), PA Drvr.3 (PA_INT), PA Rb2.1 (PA_INT), PA Rb2.2 (PA_INT), PA Rc1.2 (PA_INT)
- new net PHY1_INTRN: PB2-P2.16 (PHY1_INTRN)
- new net PHY1_RSTN: PB2-P2.15 (PHY1_RSTN)
- new net PHY2_INTRN: ETH-PHY.20 (PHY2_INTRN), PB2-P2.14 (PHY2_INTRN)
- new net PHY2_RSTN: ETH-PHY.35 (PHY2_RSTN), PB2-P2.13 (PHY2_RSTN)
- new net PRU_1553_RX_N: PB2-P1.5 (PRU_1553_RX_N)
- new net PRU_1553_RX_P: PB2-P1.6 (PRU_1553_RX_P)
- new net PRU_1553_TX_N: PB2-P1.7 (PRU_1553_TX_N)
- new net PRU_1553_TX_P: PB2-P1.8 (PRU_1553_TX_P)
- new net PWM_CH0: PB2-P2.6 (PWM_CH0)
- new net PWM_CH1: PB2-P2.5 (PWM_CH1)
- new net PWM_CH2: PB2-P2.4 (PWM_CH2)
- new net PWM_CH3: PB2-P2.3 (PWM_CH3)
- new net RF_ANT_SW: T/R Sw.1 (RF_ANT_SW)
- new net RF_FILT: C3 120p.1 (RF_FILT), L3 180n.2 (RF_FILT), T/R Sw.5 (RF_FILT)
- new net RF_LPF_N1: C1 120p.1 (RF_LPF_N1), L1 100n.2 (RF_LPF_N1), L2 180n.1 (RF_LPF_N1)
- new net RF_LPF_N2: C2 180p.1 (RF_LPF_N2), L2 180n.2 (RF_LPF_N2), L3 180n.1 (RF_LPF_N2)
- new net RF_RX: LNA.3 (RF_RX), T/R Sw.3 (RF_RX)
- new net RF_TX: ANT TVS.5 (RF_TX), L1 100n.1 (RF_TX), PA 100mW.3 (RF_TX), PA By2.1 (RF_TX)
- new net RMII0_CRS_DV: PB2-P2.29 (RMII0_CRS_DV)
- new net RMII0_REF_CLK: PB2-P2.27 (RMII0_REF_CLK)
- new net RMII0_RXD0: PB2-P2.31 (RMII0_RXD0)
- new net RMII0_RXD1: PB2-P2.30 (RMII0_RXD1)
- new net RMII0_RX_ER: PB2-P2.28 (RMII0_RX_ER)
- new net RMII0_TXD0: PB2-P2.34 (RMII0_TXD0)
- new net RMII0_TXD1: PB2-P2.33 (RMII0_TXD1)
- new net RMII0_TX_EN: PB2-P2.32 (RMII0_TX_EN)
- new net RMII1_CRS_DV: ETH-PHY.32 (RMII1_CRS_DV), PB2-P2.21 (RMII1_CRS_DV)
- new net RMII1_REF_CLK: ETH-PHY.29 (RMII1_REF_CLK), PB2-P2.19 (RMII1_REF_CLK)
- new net RMII1_RXD0: ETH-PHY.30 (RMII1_RXD0), PB2-P2.23 (RMII1_RXD0)
- new net RMII1_RXD1: ETH-PHY.31 (RMII1_RXD1), PB2-P2.22 (RMII1_RXD1)
- new net RMII1_RX_ER: ETH-PHY.33 (RMII1_RX_ER), PB2-P2.20 (RMII1_RX_ER)
- new net RMII1_TXD0: ETH-PHY.28 (RMII1_TXD0), PB2-P2.26 (RMII1_TXD0)
- new net RMII1_TXD1: ETH-PHY.27 (RMII1_TXD1), PB2-P2.25 (RMII1_TXD1)
- new net RMII1_TX_EN: ETH-PHY.26 (RMII1_TX_EN), PB2-P2.24 (RMII1_TX_EN)
- new net RS485_DE: PB2-P1.9 (RS485_DE)
- new net RS485_RX: PB2-P1.10 (RS485_RX)
- new net RS485_TX: PB2-P1.11 (RS485_TX)
- new net RSSI_ANA: RSSI Hi.2 (RSSI_ANA), RSSI Lo.1 (RSSI_ANA), RSSI_CMP.1 (RSSI_ANA)
- new net RSSI_DCD: PB2-P2.2 (RSSI_DCD), RSSI_CMP.5 (RSSI_DCD)
- new net RSSI_RAW: LNA.2 (RSSI_RAW), RSSI Hi.1 (RSSI_RAW)
- new net RSSI_REF: RSSI_CMP.3 (RSSI_REF), RSSI_RH.2 (RSSI_REF), RSSI_RL.1 (RSSI_REF)
- new net RX_LNA: 1.2k R.1 (RX_LNA), 2.2k R.1 (RX_LNA), LNA.1 (RX_LNA)
- new net SBUS_OUT: INV1.3 (SBUS_OUT), MUX1.6 (SBUS_OUT)
- new net SDIO_CLK: PB2-P1.32 (SDIO_CLK)
- new net SDIO_CMD: PB2-P1.31 (SDIO_CMD)
- new net SDIO_D0: PB2-P1.30 (SDIO_D0)
- new net SDIO_D1: PB2-P1.29 (SDIO_D1)
- new net SDIO_D2: PB2-P1.28 (SDIO_D2)
- new net SDIO_D3: PB2-P1.27 (SDIO_D3)
- new net SPI1_CLK: LoRa.4 (SPI1_CLK), PB2-P1.25 (SPI1_CLK)
- new net SPI1_CS_LORA: LoRa.5 (SPI1_CS_LORA), PB2-P1.26 (SPI1_CS_LORA)
- new net SPI1_CS_NOR: PB2-P1.22 (SPI1_CS_NOR)
- new net SPI1_CS_TPM: PB2-P1.21 (SPI1_CS_TPM)
- new net SPI1_MISO: LoRa.2 (SPI1_MISO), PB2-P1.23 (SPI1_MISO)
- new net SPI1_MOSI: LoRa.3 (SPI1_MOSI), PB2-P1.24 (SPI1_MOSI)
- new net TCXO_OUT: 49M DDS.8 (TCXO_OUT), TCXO 25M.3 (TCXO_OUT)
- new net TPM_IRQN: PB2-P2.12 (TPM_IRQN)
- new net TPM_RSTN: PB2-P2.11 (TPM_RSTN)
- new net UART_RCRS_RX: PB2-P1.15 (UART_RCRS_RX), UART CMC.1 (UART_RCRS_RX), UART TVS.2 (UART_RCRS_RX)
- new net UART_RCRS_TX: PB2-P1.16 (UART_RCRS_TX), UART CMC.4 (UART_RCRS_TX), UART TVS.5 (UART_RCRS_TX)
- new net UART_RX_F: INV1.1 (UART_RX_F), MUX1.1 (UART_RX_F), RX Bead.1 (UART_RX_F), RX Bead.2 (UART_RX_F)
- new net UART_RX_MUX: MUX1.3 (UART_RX_MUX), UART CMC.3 (UART_RX_MUX)
- new net UART_SIK_RX: PB2-P1.17 (UART_SIK_RX)
- new net UART_SIK_TX: PB2-P1.18 (UART_SIK_TX)
- new net UART_TX_F: TX Bead.1 (UART_TX_F), TX Bead.2 (UART_TX_F), UART CMC.2 (UART_TX_F)
- new net VCC2_ETH: ETH-PHY.40 (VCC2_ETH), ETH-PHY.41 (VCC2_ETH), ETH-PHY.7 (VCC2_ETH), ETH-PHY.8 (VCC2_ETH), ETH-PHY.9 (VCC2_ETH)
- new net WINCH_IN1: PB2-P2.10 (WINCH_IN1)
- new net WINCH_IN2: PB2-P2.9 (WINCH_IN2)
- no-connect marks 0 -> 26
Other:
- note added: "6-ELEMENT CHEBYSHEV LPF"
- note added: "AFSK MODEM (MCP4921 TX DAC, LM393 RX demod, tone filters)"
- note added: "DDS / TCXO (Si5351A 49 MHz synthesiser)"
- note added: "ETHERNET 2nd PORT (ADIN1300 PHY + T-ETH isolation xfmr, JST-GH-4P line)"
- note added: "LoRa 915 MHz (RFM95W, SPI via PB2-P1)"
- note added: "PA CHAIN (MMBT2222A driver + 2N3866 100 mW final)"
- note added: "PB2-I PASSTHROUGH RAILS (PocketBeagle 2 Industrial P1 + P2)"
- note added: "POWER SUPPLY (5V input filter, MCP1703 LDO, bypass cascade)"
- note added: "RSSI CARRIER-DETECT (NEW 2026-07-04 — analog RSSI -> 1-bit RSSI_DCD)"
- note added: "T/R SWITCH, LNA, ANTENNA PORT"
- note added: "UART / SBUS DIGITAL (CMC, TVS, beads, inverter, mux)"
- title: XCVR-49MHZ-2 EMI-Hardened 49 MHz AX.25 KISS Transceiver -> Emma — 49 MHz AX.25 + LoRa 915 MHz Transceiver Cape (Rev S1)
