File: kicad/Vera.kicad_pcb (KiCad board)
At the start: 4 copper layers, 69.8 x 56.4 mm, 45 parts, among them Q1 AO3400, T1 Wurth 749010012A, T2 Wurth 749010012A, U1 TI AM62A7, U2 Microchip KSZ9477, U3 TI MSPM0G3507, U4 TI ISOW1044BDFMR, U5 Infineon SLB9670, Y1 25MHz

Commit message: reorg and fixes
Parts:
- removed H1, H2, H3, H4: M3, MountingHole:MountingHole_3.2mm_M3
- U_SOM: moved to B.Cu
- moved J_PWR 225.7 mm to (179.0, 170.0)
- moved J_ETH_OUT 223.6 mm to (178.0, 159.5), turned to 90 degrees
- moved J_LASER 222.6 mm to (239.0, 150.0)
- moved C_ISO 222.4 mm to (225.9, 143.1)
- moved MH1 222.4 mm to (240.7, 141.0)
- moved MH2 222.4 mm to (240.7, 161.6)
- moved MH3 222.4 mm to (176.9, 176.5)
- moved MH4 222.4 mm to (176.9, 126.1)
- moved U_SOM 222.4 mm to (197.9, 151.3)
- moved Q1 222.4 mm to (226.9, 159.1)
- moved J_CAM_DS 221.4 mm to (237.5, 156.5)
- moved T2 219.6 mm to (188.3, 159.5), turned to -90 degrees
- moved J_ETH_IN 219.2 mm to (178.0, 147.5), turned to 90 degrees
- moved J_CHASSIS_R 218.5 mm to (226.0, 140.5)
- moved U4 218.5 mm to (225.0, 151.0)
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