File: kicad/Jayne/kicads/Jayne.kicad_pcb (KiCad board)
At the start: 4 copper layers, 69.8 x 56.4 mm, 63 parts, among them Q1 AO3400 logic-level N-MOSFET, T1 Wurth 749010012A, T1_CMC1 SRF2012-100Y, T1_CMC2 SRF2012-100Y, T1_D1 PRTR5V0U2X, T1_D2 PRTR5V0U2X, T2 Wurth 749010012A, T2_CMC1 SRF2012-100Y, T2_CMC2 SRF2012-100Y, T2_D1 PRTR5V0U2X, T2_D2 PRTR5V0U2X, U2 Microchip KSZ9477, U3 TI MSPM0G3507, U4 TI ISOW1044BDFMR, U5 Infineon SLB9670, Y1 25MHz

Commit message: fixed wash and jayne
Parts:
- T1, T2: moved to B.Cu
- moved Y1 79.6 mm to (184.2, 130.0)
- moved U_REG_3V3_CO 68.7 mm to (213.1, 151.5)
- moved R_FB3T 68.1 mm to (213.0, 149.5)
- moved J_PWR 67.5 mm to (178.6, 132.1), turned to 90 degrees
- moved U_REG_1V2_CI 65.9 mm to (213.0, 147.5)
- moved U_REG_2V5 64.6 mm to (216.4, 147.1), turned to 90 degrees
- moved J_CHASSIS_R 63.9 mm to (212.6, 146.0)
- moved R_ISET 63.2 mm to (213.5, 154.0)
- moved T2_D1 62.0 mm to (216.2, 142.4), turned to 90 degrees
- moved Q1 61.5 mm to (228.9, 152.6)
- moved R_NRST 61.0 mm to (213.5, 155.5)
- moved R1 59.6 mm to (217.9, 150.5)
- moved R2 59.6 mm to (220.5, 150.5)
- moved R_FB1B 59.6 mm to (223.0, 150.5)
- moved U_REG_3V3_CI 58.1 mm to (209.5, 163.0)
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
Commit message: changed avionics names to non ip sensitive names
Parts:
- J_CAM_DS: footprint Jayne:DS_Camera_9P -> Observer:DS_Camera_9P
- J_LASER_DS: footprint Jayne:DS_Laser_2P -> Observer:DS_Laser_2P
- J_TOF_DS: footprint Jayne:DS_ToF_4P -> Observer:DS_ToF_4P
- T1, T2: footprint Jayne:Wurth_749010012A_10-100BASE-TX -> Observer:Wurth_749010012A_10-100BASE-TX
- U2: footprint Jayne:TQFP-128-1EP_KSZ9477_14x14mm_P0.4mm_EP10x10 -> Observer:TQFP-128-1EP_KSZ9477_14x14mm_P0.4mm_EP10x10
- U_SOM: footprint Jayne:phyCORE-AM62x_PCM071_2xBTH-060 -> Observer:phyCORE-AM62x_PCM071_2xBTH-060
Other:
- board text added: "Observer Rev - (design exploration)"
- board text removed: "Jayne Rev - (design exploration)"
Changed lines of the file:
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@@
 	(paper "A3")
 	(title_block
-		(title "Jayne — Nose/Cargo-Bay Vision, ToF & Laser Board (Jayne cargo-handling system)")
+		(title "Observer — Nose/Cargo-Bay Vision, ToF & Laser Board (Observer cargo-handling system)")
 		(date "2026-07-03")
 		(rev "-")
@@
 	(net 91 "U_REG_3V3_FB")
 	(net 92 "U_REG_3V3_SW")
-	(footprint "Jayne:TQFP-128-1EP_KSZ9477_14x14mm_P0.4mm_EP10x10"
+	(footprint "Observer:TQFP-128-1EP_KSZ9477_14x14mm_P0.4mm_EP10x10"
 		(layer "F.Cu")
 		(at 192.5 140.5)
@@
 		)
 	)
-	(footprint "Jayne:DS_Camera_9P"
+	(footprint "Observer:DS_Camera_9P"
 		(layer "F.Cu")
 		(at 230 148.5)
@@
 		)
 	)
-	(footprint "Jayne:DS_Laser_2P"
+	(footprint "Observer:DS_Laser_2P"
 		(layer "F.Cu")
 		(at 233.5 153)
@@
 		)
 	)
-	(footprint "Jayne:DS_ToF_4P"
+	(footprint "Observer:DS_ToF_4P"
 		(layer "F.Cu")
 		(at 224.5 162)
@@
 		(embedded_fonts no)
 	)
-	(footprint "Jayne:Wurth_749010012A_10-100BASE-TX"
+	(footprint "Observer:Wurth_749010012A_10-100BASE-TX"
 		(layer "B.Cu")
 		(at 229 146.5 180)
@@
 		(embedded_fonts no)
 	)
-	(footprint "Jayne:phyCORE-AM62x_PCM071_2xBTH-060"
+	(footprint "Observer:phyCORE-AM62x_PCM071_2xBTH-060"
 		(layer "B.Cu")
 		(at 200 151 90)
@@
 		(embedded_fonts no)
 	)
-	(footprint "Jayne:Wurth_749010012A_10-100BASE-TX"
+	(footprint "Observer:Wurth_749010012A_10-100BASE-TX"
 		(layer "B.Cu")
 		(at 229 156.27)
@@
 		(layer "Edge.Cuts")
 	)
-	(gr_text "Jayne Rev - (design exploration)"
+	(gr_text "Observer Rev - (design exploration)"
 		(at 22.5 39.5 -0)
 		(layer "B.Fab")
