File: kicad/Jayne/kicads/Jayne.kicad_sch (KiCad schematic)
At the start: 59 parts, among them Q1 AO3400 logic-level N-MOSFET, T1 Wurth 749010012A, T1_CMC1 SRF2012-100Y, T1_CMC2 SRF2012-100Y, T1_D1 PRTR5V0U2X, T1_D2 PRTR5V0U2X, T2 Wurth 749010012A, T2_CMC1 SRF2012-100Y, T2_CMC2 SRF2012-100Y, T2_D1 PRTR5V0U2X, T2_D2 PRTR5V0U2X, U2 Microchip KSZ9477, U3 TI MSPM0G3507, U4 TI ISOW1044BDFMR, U5 Infineon SLB9670, Y1 25MHz

Commit message: changed avionics names to non ip sensitive names
Parts:
- J_CAM_DS: footprint Jayne:DS_Camera_9P -> Observer:DS_Camera_9P
- J_LASER_DS: footprint Jayne:DS_Laser_2P -> Observer:DS_Laser_2P
- J_TOF_DS: footprint Jayne:DS_ToF_4P -> Observer:DS_ToF_4P
- T1, T2: footprint Jayne:Wurth_749010012A_10-100BASE-TX -> Observer:Wurth_749010012A_10-100BASE-TX
- U2: footprint Jayne:TQFP-128-1EP_KSZ9477_14x14mm_P0.4mm_EP10x10 -> Observer:TQFP-128-1EP_KSZ9477_14x14mm_P0.4mm_EP10x10
- U_SOM: footprint Jayne:phyCORE-AM62x_PCM071_2xBTH-060 -> Observer:phyCORE-AM62x_PCM071_2xBTH-060
Other:
- title: Jayne — Nose/Cargo-Bay Vision, ToF & Laser Board (SoM end-state) -> Observer — Nose/Cargo-Bay Vision, ToF & Laser Board (SoM end-state)
Changed lines of the file:
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@@
   (paper "A1")
   (title_block
-    (title "Jayne — Nose/Cargo-Bay Vision, ToF & Laser Board (SoM end-state)") (date "2026-07-13") (rev "S1") (company "Griffing Technology LLC")
+    (title "Observer — Nose/Cargo-Bay Vision, ToF & Laser Board (SoM end-state)") (date "2026-07-13") (rev "S1") (company "Griffing Technology LLC")
     (comment 1 "Serenity UAV — STANDALONE board, NOT a PocketBeagle 2 Industrial cape")
     (comment 2 "Copyright 2026 Steve Griffing PE(CSE) CISSP-ISSEP CPP | Griffing Technology LLC")
@@
     (property "Value" "phyCORE-AM62x PCM-071" (at 185.42 92.17 0)
       (effects (font (size 1.27 1.27))))
-    (property "Footprint" "Jayne:phyCORE-AM62x_PCM071_2xBTH-060" (at 0 0 0)
+    (property "Footprint" "Observer:phyCORE-AM62x_PCM071_2xBTH-060" (at 0 0 0)
       (effects (font (size 1.27 1.27)) (hide yes)))
   )
@@
     (property "Value" "phyCORE-AM62x PCM-071" (at 255.27 92.17 0)
       (effects (font (size 1.27 1.27))))
-    (property "Footprint" "Jayne:phyCORE-AM62x_PCM071_2xBTH-060" (at 0 0 0)
+    (property "Footprint" "Observer:phyCORE-AM62x_PCM071_2xBTH-060" (at 0 0 0)
       (effects (font (size 1.27 1.27)) (hide yes)))
   )
@@
     (property "Value" "phyCORE-AM62x PCM-071" (at 325.12 92.17 0)
       (effects (font (size 1.27 1.27))))
-    (property "Footprint" "Jayne:phyCORE-AM62x_PCM071_2xBTH-060" (at 0 0 0)
+    (property "Footprint" "Observer:phyCORE-AM62x_PCM071_2xBTH-060" (at 0 0 0)
       (effects (font (size 1.27 1.27)) (hide yes)))
   )
@@
     (property "Value" "phyCORE-AM62x PCM-071" (at 394.97 92.17 0)
       (effects (font (size 1.27 1.27))))
-    (property "Footprint" "Jayne:phyCORE-AM62x_PCM071_2xBTH-060" (at 0 0 0)
+    (property "Footprint" "Observer:phyCORE-AM62x_PCM071_2xBTH-060" (at 0 0 0)
       (effects (font (size 1.27 1.27)) (hide yes)))
   )
@@
     (property "Value" "Microchip KSZ9477" (at 180.34 252.19 0)
       (effects (font (size 1.27 1.27))))
-    (property "Footprint" "Jayne:TQFP-128-1EP_KSZ9477_14x14mm_P0.4mm_EP10x10" (at 0 0 0)
+    (property "Footprint" "Observer:TQFP-128-1EP_KSZ9477_14x14mm_P0.4mm_EP10x10" (at 0 0 0)
       (effects (font (size 1.27 1.27)) (hide yes)))
   )
@@
     (property "Value" "Microchip KSZ9477" (at 240.03 252.19 0)
       (effects (font (size 1.27 1.27))))
-    (property "Footprint" "Jayne:TQFP-128-1EP_KSZ9477_14x14mm_P0.4mm_EP10x10" (at 0 0 0)
+    (property "Footprint" "Observer:TQFP-128-1EP_KSZ9477_14x14mm_P0.4mm_EP10x10" (at 0 0 0)
       (effects (font (size 1.27 1.27)) (hide yes)))
   )
@@
     (property "Value" "Microchip KSZ9477" (at 299.72 252.19 0)
       (effects (font (size 1.27 1.27))))
-    (property "Footprint" "Jayne:TQFP-128-1EP_KSZ9477_14x14mm_P0.4mm_EP10x10" (at 0 0 0)
+    (property "Footprint" "Observer:TQFP-128-1EP_KSZ9477_14x14mm_P0.4mm_EP10x10" (at 0 0 0)
       (effects (font (size 1.27 1.27)) (hide yes)))
   )
@@
     (property "Value" "Microchip KSZ9477" (at 359.41 252.19 0)
       (effects (font (size 1.27 1.27))))
-    (property "Footprint" "Jayne:TQFP-128-1EP_KSZ9477_14x14mm_P0.4mm_EP10x10" (at 0 0 0)
+    (property "Footprint" "Observer:TQFP-128-1EP_KSZ9477_14x14mm_P0.4mm_EP10x10" (at 0 0 0)
       (effects (font (size 1.27 1.27)) (hide yes)))
   )
@@
     (property "Value" "Microchip KSZ9477" (at 430.53 252.19 0)
       (effects (font (size 1.27 1.27))))
-    (property "Footprint" "Jayne:TQFP-128-1EP_KSZ9477_14x14mm_P0.4mm_EP10x10" (at 0 0 0)
+    (property "Footprint" "Observer:TQFP-128-1EP_KSZ9477_14x14mm_P0.4mm_EP10x10" (at 0 0 0)
       (effects (font (size 1.27 1.27)) (hide yes)))
   )
@@
     (property "Value" "Microchip KSZ9477" (at 485.14 252.19 0)
       (effects (font (size 1.27 1.27))))
-    (property "Footprint" "Jayne:TQFP-128-1EP_KSZ9477_14x14mm_P0.4mm_EP10x10" (at 0 0 0)
+    (property "Footprint" "Observer:TQFP-128-1EP_KSZ9477_14x14mm_P0.4mm_EP10x10" (at 0 0 0)
       (effects (font (size 1.27 1.27)) (hide yes)))
   )
@@
     (property "Value" "Wurth 749010012A" (at 250.00 333.81 0)
       (effects (font (size 1.27 1.27))))
-    (property "Footprint" "Jayne:Wurth_749010012A_10-100BASE-TX" (at 0 0 0)
+    (property "Footprint" "Observer:Wurth_749010012A_10-100BASE-TX" (at 0 0 0)
       (effects (font (size 1.27 1.27)) (hide yes)))
     (property "Datasheet" "" (at 0 0 0)
@@
     (property "Value" "Wurth 749010012A" (at 250.00 373.81 0)
       (effects (font (size 1.27 1.27))))
-    (property "Footprint" "Jayne:Wurth_749010012A_10-100BASE-TX" (at 0 0 0)
+    (property "Footprint" "Observer:Wurth_749010012A_10-100BASE-TX" (at 0 0 0)
       (effects (font (size 1.27 1.27)) (hide yes)))
     (property "Datasheet" "" (at 0 0 0)
@@
     (property "Value" "Direct-solder camera land (nose; DNP if J_CAM* used)" (at 320.00 448.81 0)
       (effects (font (size 1.27 1.27))))
-    (property "Footprint" "Jayne:DS_Camera_9P" (at 0 0 0)
+    (property "Footprint" "Observer:DS_Camera_9P" (at 0 0 0)
       (effects (font (size 1.27 1.27)) (hide yes)))
     (property "Datasheet" "" (at 0 0 0)
@@
     (property "Value" "Direct-solder ToF land (nose; DNP if J_TOF used)" (at 285.00 483.81 0)
       (effects (font (size 1.27 1.27))))
-    (property "Footprint" "Jayne:DS_ToF_4P" (at 0 0 0)
+    (property "Footprint" "Observer:DS_ToF_4P" (at 0 0 0)
       (effects (font (size 1.27 1.27)) (hide yes)))
     (property "Datasheet" "" (at 0 0 0)
@@
     (property "Value" "Direct-solder laser land (nose; DNP if J_LASER used)" (at 410.00 483.81 0)
       (effects (font (size 1.27 1.27))))
-    (property "Footprint" "Jayne:DS_Laser_2P" (at 0 0 0)
-      (effects (font (size 1.27 1.27)) (hide yes)))
-    (property "Datasheet" "" (at 0 0 0)
+    (property "Footprint" "Observer:DS_Laser_2P" (at 0 0 0)
+      (effects (font (size 1.27 1.27)) (hide yes)))
+    (property "Datasheet" "" (at 0 0 0)
