File: kicad/Kaylee/kicads/Kaylee.kicad_pcb (KiCad board)
At the start: 4 copper layers, 90 x 65 mm, 67 parts

Commit message: changed avionics names to non ip sensitive names
Parts:
- CM1, CM2: footprint Kaylee:CMC_WE-SL5_7440640500 -> FlightEngineer:CMC_WE-SL5_7440640500
- F1: footprint Kaylee:FuseHolder_MAXI_PCB -> FlightEngineer:FuseHolder_MAXI_PCB
- RS_1, RS_2, RS_3, RS_4, RS_MAIN: footprint Kaylee:R_Shunt_CSS2H_2512K -> FlightEngineer:R_Shunt_CSS2H_2512K
Other:
- board text added: "FlightEngineer Rev R"
- board text removed: "Kaylee Rev R"
Changed lines of the file:
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@@
 	(paper "A4")
 	(title_block
-		(title "Kaylee")
+		(title "FlightEngineer")
 		(date "2026-06-10")
 		(rev "A")
@@
 		(stroke (width 0.05) (type default)) (layer "Edge.Cuts")
 )
-	(gr_text "Kaylee Rev R" (at 45.00 68.00 0) (layer "F.Fab")
+	(gr_text "FlightEngineer Rev R" (at 45.00 68.00 0) (layer "F.Fab")
 		(effects (font (size 1.5 1.5) (thickness 0.15)))
 )
@@
 		(pad "2" thru_hole circle (at 7.2000 0.0000) (size 4.0000 4.0000) (drill 2.5000) (layers "*.Cu" "*.Mask") (net 2 "PGND"))
 	)
-	(footprint "Kaylee:CMC_WE-SL5_7440640500" (layer "F.Cu")
+	(footprint "FlightEngineer:CMC_WE-SL5_7440640500" (layer "F.Cu")
 		(at 31.0000 12.0000)
 		(property "Reference" "CM1" (at 0 -3.5 0) (layer "F.SilkS")
@@
 		(property "Value" "WE-SL5_7440640500" (at 0 3.5 0) (layer "F.Fab")
 			(effects (font (size 1.0 1.0) (thickness 0.15))))
-		(property "Footprint" "Kaylee:CMC_WE-SL5_7440640500" (at 0 0 0) (layer "F.Fab")
+		(property "Footprint" "FlightEngineer:CMC_WE-SL5_7440640500" (at 0 0 0) (layer "F.Fab")
 			(effects (font (size 1.0 1.0) (thickness 0.15)) (hide yes)))
 		(fp_rect (start -5.5400 -5.5400) (end 5.5400 5.5400) (layer "F.CrtYd") (stroke (width 0.05) (type default)))
@@
 		(pad "4" thru_hole circle (at -2.5400 2.5400) (size 1.9000 1.9000) (drill 1.2000) (layers "*.Cu" "*.Mask") (net 2 "PGND"))
 	)
-	(footprint "Kaylee:CMC_WE-SL5_7440640500" (layer "F.Cu")
+	(footprint "FlightEngineer:CMC_WE-SL5_7440640500" (layer "F.Cu")
 		(at 44.0000 12.0000)
 		(property "Reference" "CM2" (at 0 -3.5 0) (layer "F.SilkS")
@@
 		(property "Value" "WE-SL5_7440640500" (at 0 3.5 0) (layer "F.Fab")
 			(effects (font (size 1.0 1.0) (thickness 0.15))))
-		(property "Footprint" "Kaylee:CMC_WE-SL5_7440640500" (at 0 0 0) (layer "F.Fab")
+		(property "Footprint" "FlightEngineer:CMC_WE-SL5_7440640500" (at 0 0 0) (layer "F.Fab")
 			(effects (font (size 1.0 1.0) (thickness 0.15)) (hide yes)))
 		(fp_rect (start -5.5400 -5.5400) (end 5.5400 5.5400) (layer "F.CrtYd") (stroke (width 0.05) (type default)))
@@
 		(pad "4" thru_hole circle (at -2.5400 2.5400) (size 1.9000 1.9000) (drill 1.2000) (layers "*.Cu" "*.Mask") (net 2 "PGND"))
 	)
-	(footprint "Kaylee:FuseHolder_MAXI_PCB" (layer "F.Cu")
+	(footprint "FlightEngineer:FuseHolder_MAXI_PCB" (layer "F.Cu")
 		(at 56.0000 9.0000)
 		(property "Reference" "F1" (at 0 -3.5 0) (layer "F.SilkS")
@@
 		(property "Value" "FuseHolder_MAXI_150A" (at 0 3.5 0) (layer "F.Fab")
 			(effects (font (size 1.0 1.0) (thickness 0.15))))
-		(property "Footprint" "Kaylee:FuseHolder_MAXI_PCB" (at 0 0 0) (layer "F.Fab")
+		(property "Footprint" "FlightEngineer:FuseHolder_MAXI_PCB" (at 0 0 0) (layer "F.Fab")
 			(effects (font (size 1.0 1.0) (thickness 0.15)) (hide yes)))
 		(fp_rect (start -2.2000 -7.5000) (end 12.1000 7.5000) (layer "F.CrtYd") (stroke (width 0.05) (type default)))
@@
 		(pad "2" smd roundrect (at 0.5100 0.0000) (size 0.5400 0.6400) (layers "F.Cu" "F.Mask" "F.Paste") (roundrect_rratio 0.25) (net 18 "CHASSIS"))
 	)
-	(footprint "Kaylee:R_Shunt_CSS2H_2512K" (layer "F.Cu")
+	(footprint "FlightEngineer:R_Shunt_CSS2H_2512K" (layer "F.Cu")
 		(at 39.0000 33.0000)
 		(property "Reference" "RS_MAIN" (at 0 -3.5 0) (layer "F.SilkS")
@@
 		(property "Value" "1mOhm_Kelvin_2512" (at 0 3.5 0) (layer "F.Fab")
 			(effects (font (size 1.0 1.0) (thickness 0.15))))
-		(property "Footprint" "Kaylee:R_Shunt_CSS2H_2512K" (at 0 0 0) (layer "F.Fab")
+		(property "Footprint" "FlightEngineer:R_Shunt_CSS2H_2512K" (at 0 0 0) (layer "F.Fab")
 			(effects (font (size 1.0 1.0) (thickness 0.15)) (hide yes)))
 		(attr smd)
@@
 		(pad "2" thru_hole circle (at 9.9200 3.4000) (size 2.7800 2.7800) (drill 1.7800) (layers "*.Cu" "*.Mask") (net 34 "ESC1_FUSED"))
 	)
-	(footprint "Kaylee:R_Shunt_CSS2H_2512K" (layer "F.Cu")
+	(footprint "FlightEngineer:R_Shunt_CSS2H_2512K" (layer "F.Cu")
 		(at 8.0000 47.0000)
 		(property "Reference" "RS_1" (at 0 -3.5 0) (layer "F.SilkS")
@@
 		(property "Value" "1mOhm_Kelvin_2512" (at 0 3.5 0) (layer "F.Fab")
 			(effects (font (size 1.0 1.0) (thickness 0.15))))
-		(property "Footprint" "Kaylee:R_Shunt_CSS2H_2512K" (at 0 0 0) (layer "F.Fab")
+		(property "Footprint" "FlightEngineer:R_Shunt_CSS2H_2512K" (at 0 0 0) (layer "F.Fab")
 			(effects (font (size 1.0 1.0) (thickness 0.15)) (hide yes)))
 		(attr smd)
@@
 		(pad "2" thru_hole circle (at 9.9200 3.4000) (size 2.7800 2.7800) (drill 1.7800) (layers "*.Cu" "*.Mask") (net 35 "ESC2_FUSED"))
 	)
-	(footprint "Kaylee:R_Shunt_CSS2H_2512K" (layer "F.Cu")
+	(footprint "FlightEngineer:R_Shunt_CSS2H_2512K" (layer "F.Cu")
 		(at 22.0000 47.0000)
 		(property "Reference" "RS_2" (at 0 -3.5 0) (layer "F.SilkS")
@@
 		(property "Value" "1mOhm_Kelvin_2512" (at 0 3.5 0) (layer "F.Fab")
 			(effects (font (size 1.0 1.0) (thickness 0.15))))
-		(property "Footprint" "Kaylee:R_Shunt_CSS2H_2512K" (at 0 0 0) (layer "F.Fab")
+		(property "Footprint" "FlightEngineer:R_Shunt_CSS2H_2512K" (at 0 0 0) (layer "F.Fab")
 			(effects (font (size 1.0 1.0) (thickness 0.15)) (hide yes)))
 		(attr smd)
@@
 		(pad "2" thru_hole circle (at 9.9200 3.4000) (size 2.7800 2.7800) (drill 1.7800) (layers "*.Cu" "*.Mask") (net 36 "ESC3_FUSED"))
 	)
-	(footprint "Kaylee:R_Shunt_CSS2H_2512K" (layer "F.Cu")
+	(footprint "FlightEngineer:R_Shunt_CSS2H_2512K" (layer "F.Cu")
 		(at 36.0000 47.0000)
 		(property "Reference" "RS_3" (at 0 -3.5 0) (layer "F.SilkS")
@@
 		(property "Value" "1mOhm_Kelvin_2512" (at 0 3.5 0) (layer "F.Fab")
 			(effects (font (size 1.0 1.0) (thickness 0.15))))
-		(property "Footprint" "Kaylee:R_Shunt_CSS2H_2512K" (at 0 0 0) (layer "F.Fab")
+		(property "Footprint" "FlightEngineer:R_Shunt_CSS2H_2512K" (at 0 0 0) (layer "F.Fab")
 			(effects (font (size 1.0 1.0) (thickness 0.15)) (hide yes)))
 		(attr smd)
@@
 		(pad "2" thru_hole circle (at 9.9200 3.4000) (size 2.7800 2.7800) (drill 1.7800) (layers "*.Cu" "*.Mask") (net 37 "ESC4_FUSED"))
 	)
-	(footprint "Kaylee:R_Shunt_CSS2H_2512K" (layer "F.Cu")
+	(footprint "FlightEngineer:R_Shunt_CSS2H_2512K" (layer "F.Cu")
 		(at 50.0000 47.0000)
 		(property "Reference" "RS_4" (at 0 -3.5 0) (layer "F.SilkS")
@@
 		(property "Value" "1mOhm_Kelvin_2512" (at 0 3.5 0) (layer "F.Fab")
 			(effects (font (size 1.0 1.0) (thickness 0.15))))
-		(property "Footprint" "Kaylee:R_Shunt_CSS2H_2512K" (at 0 0 0) (layer "F.Fab")
-			(effects (font (size 1.0 1.0) (thickness 0.15)) (hide yes)))
-		(attr smd)
+		(property "Footprint" "FlightEngineer:R_Shunt_CSS2H_2512K" (at 0 0 0) (layer "F.Fab")
+			(effects (font (size 1.0 1.0) (thickness 0.15)) (hide yes)))
+		(attr smd)
