File: kicad/Kaylee/kicads/Kaylee.kicad_sch (KiCad schematic)
At the start: 99 parts

Commit message: changed avionics names to non ip sensitive names
Other:
- title: Kaylee — EMI-Hardened Power Distribution Board -> FlightEngineer — EMI-Hardened Power Distribution Board
Changed lines of the file:
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@@
   (paper "A1")
   (title_block
-    (title "Kaylee — EMI-Hardened Power Distribution Board") (date "2026-06-10") (rev "A") (company "Griffing Technology LLC")
+    (title "FlightEngineer — EMI-Hardened Power Distribution Board") (date "2026-06-10") (rev "A") (company "Griffing Technology LLC")
     (comment 1 "Serenity UAV Power Distribution Board — 90x65mm 4-layer FR4-TG170")
     (comment 2 "Copyright 2026 Steve Griffing PE(CSE) CISSP-ISSEP CPP | Griffing Technology LLC")
