File: kicad/Zoë/kicads/Zoë.kicad_sch (KiCad schematic)
At the start: 52 parts, among them SW1 SW_DIP_x02, X2Y_CAN 4.7nF_X2Y, X2Y_RS485 4.7nF_X2Y

Commit message: changed avionics names to non ip sensitive names
Other:
- title: Zoë — EMI-Hardened Comms, Logging & Payload Cape -> TACCO — EMI-Hardened Comms, Logging & Payload Cape
Changed lines of the file:
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@@
   (paper "A1")
   (title_block
-    (title "Zoë — EMI-Hardened Comms, Logging & Payload Cape") (date "2026-06-07") (rev "3") (company "Griffing Technology LLC")
+    (title "TACCO — EMI-Hardened Comms, Logging & Payload Cape") (date "2026-06-07") (rev "3") (company "Griffing Technology LLC")
     (comment 1 "CN Node — Comms + Logging + Payload Cape for Serenity UAV")
     (comment 2 "Copyright 2026 Steve Griffing PE(CSE) CISSP-ISSEP CPP | Griffing Technology LLC")
